File: Noisemeter.sch (KiCad schematic (older format))
At the start: 57 parts, among them IC1 MCP1801, IC2 STM32_48pin, IC3 OPAMP_OS+-D, P1 USB, P2 SWD, P3 MIC2, P4 MOD, X1 32K768 12p5

Commit message: Version 1.0
Parts:
- removed L1: FERRITE, everykey:0603, symbol L
- added C?: 10n, symbol C
- added C?: 1u, symbol C
- added L?: ferrite, symbol L
- L2: value FERRITE -> 22-47u
Connections:
- net 3V3: now also C17.1
- net A3V3: now also IC2.9 (VDDA), C?.1, C?.1; no longer C17.1
- net GND: now also L?.1; no longer C18.2
- new net AGND: C18.2, C?.2, C?.2, L?.2
Other:
- moved on the sheet: C17, L2

Commit message: Fixed analog power supply
Parts:
- removed IC2: STM32_48pin, everykey:QFN-48-0.5-EP, symbol STM32_48pin
- added IC2: STM32L433Cx, symbol STM32L433Cx
- C20, C21: renamed from C?; footprint (none) -> everykey:0603
- L1: renamed from L?; footprint (none) -> everykey:0603
Connections:
- net 3V3: now also IC2.1 (VBAT), IC2.24 (VDD), IC2.36 (VDD), IC2.48 (VDD)
- net A3V3: now also IC2.9 (VDDA)
- net ADC1_7: now also IC2.12 (PA2)
- net AGND: now also C10.2, C13.2, C15.2, C19.2, IC3.2 (VSS), P3.2, IC2.8 (VSSA)
- net DAC1: now also IC2.14 (PA4)
- net DAC2: now also IC2.15 (PA5)
- net EN: now also IC2.41 (PB5)
- net GND: now also IC2.23 (VSS), IC2.35 (VSS), IC2.47 (VSS), IC2.PAD (VSS); no longer C10.2, C13.2, C15.2, C19.2, IC3.2 (VSS), P3.2
- net ID1: now also IC2.45 (PB8)
- net ID2: now also IC2.46 (PB9)
- net OPAMP+: now also IC2.10 (PA0)
- net OPAMP-: now also IC2.11 (PA1)
- net OPAMPOUT: now also IC2.13 (PA3)
- net SAI_FS: now also IC2.30 (PA9)
- net SAI_SCK: now also IC2.29 (PA8)
- net SAI_SD: now also IC2.31 (PA10)
- net SCL: now also IC2.42 (PB6)
- net SDA: now also IC2.43 (PB7)
- net SWCLK: now also IC2.37 (PA14-SWCLK)
- net SWDIO: now also IC2.34 (PA13-SWDIO)
- net SWO: now also IC2.39 (PB3-TRACESWO)
- net USB_DM: now also IC2.32 (PA11)
- net USB_DP: now also IC2.33 (PA12)
- net ~RST: now also IC2.7 (NRST)
- net at B2.2, R4.1: now also IC2.44 (BOOT0)
- net at C5.1, X1.1: now also IC2.3 (PC14-OSC32_IN)
- net at C4.1, X1.2: now also IC2.4 (PC15-OSC32_OUT)
- net at R22.2: now also IC2.28 (PB15)
Other:
- moved on the sheet: B1, B2, R3, R4

Commit message: minor changes, BOM rename
Parts:
- C12: value 10p -> 47p
- C9: value 200p -> 100p
- R11: value 0 -> 10K
- R12: value 470K -> 47K
Changed lines of the file:
@@
 P 3550 3700
 F 0 "C9" H 3600 3750 50  0000 L CNN
-F 1 "200p" H 3600 3650 50  0000 L CNN
+F 1 "100p" H 3600 3650 50  0000 L CNN
 F 2 "everykey:0603" H 3588 3550 50  0001 C CNN
 F 3 "" H 3550 3700 50  0000 C CNN
@@
 P 4100 6250
 F 0 "R12" H 4100 6179 60  0000 C CNN
-F 1 "470K" H 4100 6314 60  0000 C CNN
+F 1 "47K" H 4100 6314 60  0000 C CNN
 F 2 "everykey:0603" H 4100 6250 60  0001 C CNN
 F 3 "" H 4100 6250 60  0000 C CNN
@@
 P 4100 6450
 F 0 "C12" H 4125 6550 50  0000 L CNN
-F 1 "10p" H 4125 6350 50  0000 L CNN
+F 1 "47p" H 4125 6350 50  0000 L CNN
 F 2 "everykey:0603" H 4138 6300 50  0001 C CNN
 F 3 "" H 4100 6450 50  0000 C CNN
@@
 P 3500 6000
 F 0 "R11" H 3500 5929 50  0000 C CNN
-F 1 "0" H 3500 6064 50  0000 C CNN
+F 1 "10K" H 3500 6064 50  0000 C CNN
 F 2 "everykey:0603" H 3500 6000 60  0001 C CNN
 F 3 "" H 3500 6000 60  0000 C CNN
